File: comms.kicad_sch (KiCad schematic)
At the start: 10 parts, among them J6 Controller Power and RS485, U6 MAX485E

Commit message: Schematic cleanup and readme improvement.
Parts:
- C21: value 100n -> (none); footprint Capacitor_SMD:C_0805_2012Metric -> (none)
- C22: value 220p -> (none); footprint Capacitor_SMD:C_0805_2012Metric -> (none)
- J6: value Controller Power and RS485 -> (none); footprint river:TerminalBlock_KEFENG_Blue_10 -> (none)
- JP1, JP2: value ~ -> (none); footprint Connector_PinHeader_2.54mm:PinHeader_1x02_P2.54mm_Vertical -> (none)
- R19, R20, R21, R22: value 120 -> (none); footprint Resistor_SMD:R_0805_2012Metric -> (none)
- U6: value MAX485E -> (none); footprint Package_DIP:DIP-8_W7.62mm_Socket -> (none)
Other:
- note added: "RS485"
- company: (none) -> River Cat
- title: (none) -> Plant Light LED Driver
- moved on the sheet: C21, C22, J6, JP1, JP2, R19, R20, R21, R22, U6
